Commit message: minicheetah

File: resources/robots/mini_cheetah/urdf/mini_cheetah.urdf (robot description, URDF)
Before this commit: robot mini_cheetah, 15 links, 14 joints
Links:
- added link FL_foot, mass 0.15; collision sphere radius=0.015; visual sphere radius=0.015
- added link FR_foot, mass 0.15; collision sphere radius=0.015; visual sphere radius=0.015
- added link RL_foot, mass 0.15; collision sphere radius=0.015; visual sphere radius=0.015
- added link RR_foot, mass 0.15; collision sphere radius=0.015; visual sphere radius=0.015
Joints:
- added joint FL_foot_fixed: type fixed, parent FL_calf, child FL_foot, origin xyz=0 0 -0.18
- added joint FR_foot_fixed: type fixed, parent FR_calf, child FR_foot, origin xyz=0 0 -0.18
- added joint RL_foot_fixed: type fixed, parent RL_calf, child RL_foot, origin xyz=0 0 -0.18
- added joint RR_foot_fixed: type fixed, parent RR_calf, child RR_foot, origin xyz=0 0 -0.18
